File: Project_02/EAGLE/Project_02_PCB.brd (EAGLE design)
At the start: 127 x 76.2 mm, 23 parts, among them J2 F-1X03-SIP-100-32, U1 TXS0102DCTT, X1 USB-A-S

Commit message: shifted section title for header
Parts:
- removed R6: 1.5k, ENGI301:R0603
- added RC: 1.5k, ENGI301:R0603
- moved R3 57.1 mm to (48.3, 25.4)
- moved R4 19.0 mm to (67.3, 25.4)
- moved R5 19.0 mm to (86.4, 25.4)
Connections:
- net BUTTON3: now also U$5.24@P2, U$7.P$1, U$7.P$3; no longer U$3.P$1, U$3.P$3, U$5.18@P2
- net BUTTON4: now also U$5.22@P2, U$6.P$1, U$6.P$3; no longer U$4.P$1, U$4.P$3, U$5.20@P2
- net BUTTON5: now also U$4.P$1, U$4.P$3, U$5.20@P2; no longer U$5.22@P2, U$6.P$1, U$6.P$3
- net BUTTONC: now also RC.1, U$3.P$1, U$3.P$3, U$5.18@P2; no longer R6.1, U$5.24@P2, U$7.P$1, U$7.P$3
- net VDD_3P3V: now also RC.2; no longer R6.2
Routing:
- net VUSB: track 64.4 -> 0.00 mm
- net BUTTONC: track 74.7 -> 44.8 mm
- net BUTTON3: track 44.8 -> 74.7 mm
- net GND: track 113.7 -> 97.4 mm, vias 9 -> 3
- net BUTTON5: track 58.2 -> 42.4 mm
- net BUTTON4: track 42.4 -> 58.2 mm
- net VDD_5V: track 164.8 -> 175.3 mm
- added copper zone on layer 1, net VUSB
Other:
- board text added: "Multi-Fandom Kpop Fan Light with Music PCB"
- board text added: "RPL"
- board text added: "Rev. 1"
