File: Project_02/EAGLE/Project_02_PCB.sch (EAGLE design)
At the start: 23 parts, among them J2 F-1X03-SIP-100-32, U1 TXS0102DCTT, X1 USB-A-S

Commit message: updated schematic
Parts:
- removed R6: 1.5k, ENGI301:R_R0603
- added RC: 1.5k, ENGI301:R_R0603
Connections:
- net BUTTON3: now also U$5.GPIO44, U$7.1, U$7.3; no longer U$3.1, U$3.3, U$5.GPIO47
- net BUTTON4: now also U$5.GPIO46, U$6.1, U$6.3; no longer U$4.1, U$4.3, U$5.GPIO64
- net BUTTON5: now also U$4.1, U$4.3, U$5.GPIO64; no longer U$5.GPIO46, U$6.1, U$6.3
- net BUTTONC: now also RC.1, U$3.1, U$3.3, U$5.GPIO47; no longer R6.1, U$5.GPIO44, U$7.1, U$7.3
- net VDD_3P3V: now also RC.2; no longer R6.2
Other:
- moved on the sheet: J2, R4, R5
